File: hardware/sbc-rk3576/kicad/rk3576-sbc.kicad_pcb (KiCad board)
At the start: 8 copper layers, 100 x 72 mm, 484 parts, among them J1001 USB3.0 A, J101 USB-C PWR/OTG, J1301 RJ45 GbE, J1401 USB2.0 A x2, J1402 u.FL, J501 DEBUG UART, J701 microSD, J801 M.2 M-KEY, J901 HDMI, Q1301 BSS138, Q1401 BSS138, Q901 BSS138, Q902 BSS138, Q903 BSS138, Q904 BSS138, Q905 BSS138, Q906 BSS138, Q907 BSS138, SW501 MASKROM, SW502 POWER, SW503 RESET, U1001 USBLC6-2SC6, U1002 TPD4E05U06, U1003 USBLC6-2SC6, U1004 AP2171W, U1301 RTL8211F-CG, U1401 FE1.1s, U1402 USBLC6-2SC6, U1403 USBLC6-2SC6, U1404 AP2171W, U1405 BL-M8821CU1, U201 RK806S-5, U301 TPS562201, U302 TPS562201, U303 TPS562201, U304 TPS563201, U305 AP2171W, U401 RK3576, U601 LPDDR5 4GB, U701 eMMC 32GB, U702 AP2171W, U901 TPD4E05U06, U902 TPD4E05U06, Y1301 25MHz, Y1401 12MHz, Y501 24MHz

Commit message: hardware: route.py chunks stop at 1h15 with optimizer off (result always saved); test chunk 703->695
Co-Authored-By: Claude Opus 5.5 <noreply@anthropic.com>
Claude-Session: https://claude.ai/code/session_01DP7VBm9fUdwhcDWq3gWKJ6
Routing:
- net RGMII_RXC: track 0.00 -> 42.8 mm, vias 1 -> 3
- net PMIC_SW10: track 0.00 -> 21.0 mm, vias 0 -> 2
- net LP5_RDQS1N_A: track 0.00 -> 17.5 mm, vias 2 -> 4
- net VDD_CPU_LIT_S0: track 19.8 -> 33.9 mm, vias 5 -> 7
- net VBUS_IN: track 0.00 -> 11.9 mm
- net VCC5V0_SYS_S5: track 14.9 -> 22.5 mm
- net BUCK_1V1_SW: track 0.00 -> 7.39 mm
- net VDD_GPU_S0: track 2.59 -> 9.10 mm, vias 5 -> 7
- net PHY_RSET: track 25.8 -> 20.0 mm
- net ETH_MDI1_N: track 3.03 -> 1.70 mm
- net PHY_LED1: track 48.8 -> 47.8 mm
- net GND: track 513.9 -> 514.7 mm
- net VDD2H_DDR_S3: track 12.0 -> 12.7 mm
- net HDMI_SCL_5V: track 15.7 -> 15.0 mm

Commit message: hardware: routing chunk 3 imported (unrouted 695 -> 558)
Co-Authored-By: Claude Opus 5.5 <noreply@anthropic.com>
Claude-Session: https://claude.ai/code/session_01DP7VBm9fUdwhcDWq3gWKJ6
Routing:
- net ETH_MDIO: track 0.93 -> 73.1 mm, vias 2 -> 4
- net LED_SYS_A: track 4.23 -> 55.9 mm, vias 0 -> 1
- net SD_PWREN: track 0.00 -> 47.3 mm, vias 1 -> 2
- net LP5_DQ6_B: track 0.00 -> 44.0 mm
- net VDD2H_DDR_S3: track 12.7 -> 56.1 mm
- net LP5_RDQS1N_B: track 0.00 -> 35.8 mm
- net USB_OTG0_VBUSDET: track 27.5 -> 60.9 mm, vias 3 -> 4
- net SD_D3: track 29.5 -> 62.3 mm
- net PCIE0_RXN: track 0.00 -> 29.0 mm, vias 1 -> 3
- net VDDQ_DDR_S0: track 0.00 -> 26.9 mm
- net HDMI_D3_TERM: track 1.50 -> 25.7 mm, vias 0 -> 2
- net PCIE0_TXP: track 0.00 -> 24.1 mm, vias 1 -> 2
- net HDMI_D1P_C: track 23.4 -> 46.0 mm, vias 1 -> 2
- net HDMI_D0N_C: track 23.0 -> 45.4 mm, vias 0 -> 3
- net HDMI_D2_TERM: track 2.91 -> 24.5 mm, vias 0 -> 2
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