File: hardware/sbc-rk3576/kicad/rk3576-sbc.kicad_pcb (KiCad board)
At the start: 8 copper layers, 100 x 72 mm, 484 parts, among them J1001 USB3.0 A, J101 USB-C PWR/OTG, J1301 RJ45 GbE, J1401 USB2.0 A x2, J1402 u.FL, J501 DEBUG UART, J701 microSD, J801 M.2 M-KEY, J901 HDMI, Q1301 BSS138, Q1401 BSS138, Q901 BSS138, Q902 BSS138, Q903 BSS138, Q904 BSS138, Q905 BSS138, Q906 BSS138, Q907 BSS138, SW501 MASKROM, SW502 POWER, SW503 RESET, U1001 USBLC6-2SC6, U1002 TPD4E05U06, U1003 USBLC6-2SC6, U1004 AP2171W, U1301 RTL8211F-CG, U1401 FE1.1s, U1402 USBLC6-2SC6, U1403 USBLC6-2SC6, U1404 AP2171W, U1405 BL-M8821CU1, U201 RK806S-5, U301 TPS562201, U302 TPS562201, U303 TPS562201, U304 TPS563201, U305 AP2171W, U401 RK3576, U601 LPDDR5 4GB, U701 eMMC 32GB, U702 AP2171W, U901 TPD4E05U06, U902 TPD4E05U06, Y1301 25MHz, Y1401 12MHz, Y501 24MHz

Commit message: hardware: board at 72 open connections, DRC clean
Slow nets routed across the power layers and pours re-planned around
them (pour_fix): 78 -> 72 open, 0 DRC errors besides them, ERC 0,
parity 0. Fab drafts, renders, length report, README and LOG #32 updated.

Co-Authored-By: Claude Opus 5.5 <noreply@anthropic.com>
Claude-Session: https://claude.ai/code/session_01DP7VBm9fUdwhcDWq3gWKJ6
Routing:
- net VCCA_1V8_S0: track 102.3 -> 154.0 mm, vias 40 -> 44
- net VDD_0V75_S3: track 57.2 -> 105.6 mm, vias 19 -> 25
- net VDD_NPU_S0: track 43.0 -> 87.3 mm, vias 28 -> 33
- net VDD_CPU_LIT_S0: track 83.3 -> 125.1 mm
- net WIFI_PD_GPIO: track 4.13 -> 44.7 mm, vias 1 -> 5
- net SD_DET_L: track 4.48 -> 44.5 mm, vias 1 -> 3
- net VCC_1V8_S3: track 77.3 -> 117.1 mm, vias 42 -> 43
- net VDDA_0V85_S0: track 42.3 -> 80.6 mm
- net VDDA0V75_HDMI_S0: track 21.0 -> 59.2 mm, vias 11 -> 13
- net PHY_INT_L: track 8.55 -> 46.6 mm, vias 3 -> 8
- net VCCA_3V3_S0: track 23.5 -> 61.5 mm
- net DBG_UART_TX: track 0.00 -> 34.6 mm, vias 1 -> 3
- net PCIE0_WAKE_L: track 9.83 -> 43.2 mm, vias 1 -> 5
- net VCC_1V1_NLDO_S3: track 85.9 -> 117.4 mm, vias 18 -> 24
- net VDDA_1V2_S0: track 2.38 -> 31.1 mm, vias 4 -> 5
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- added copper zone on In6.Cu, net VCCA_3V3_S0
- added copper zone on In6.Cu, net VDDA_0V75_S0
- added copper zone on In6.Cu, net VDDA_DDR_PLL_S0
- added copper zone on In6.Cu, net VDDQ_DDR_S0
- added copper zone on In6.Cu, net VDD_0V75_S3
