File: hardware/sbc-rk3576/kicad/02_pmic.kicad_sch (KiCad schematic)
At the start: 77 parts, among them U201 RK806S-5

Commit message: hardware: fix RK806 rail map (verified vs mainline DTS); add board device tree + Linux PC report
- RK806S-5 dcdc1-10 / nldo1-5 -> rail assignments now match mainline
  rk3576-rock-4d.dts (same PMIC OTP + SoC); rev A0 had 12 wrong.
- software/rk3576-sbc.dts compiles against mainline rk3576.dtsi
  (tools/check_dts.sh); all 7 DT GPIOs cross-checked with design.py nets.
- docs/linux_pc_readiness.md, length_report.py, route.py (Freerouting).

Co-Authored-By: Claude Opus 5.5 <noreply@anthropic.com>
Claude-Session: https://claude.ai/code/session_01DP7VBm9fUdwhcDWq3gWKJ6
Connections:
- net VCC_1V8_S3: now also C229.1, C230.1, L208.2, U201.5 (VOUT8); no longer C232.1, C233.1, L209.2, R209.2, U201.67 (VOUT9)
- net VCC_3V3_S3: now also C216.1, C217.1, C218.1, L204.2, U201.24 (VOUT4); no longer C226.1, C227.1, L207.2, U201.41 (VOUT7)
- net VDD2H_DDR_S3: now also C232.1, C233.1, L209.2, R209.2, U201.67 (VOUT9); no longer C229.1, C230.1, L208.2, U201.5 (VOUT8)
- net VDDA0V75_HDMI_S0: now also C239.1, U201.11 (NLDO3); no longer C238.1, U201.10 (NLDO4)
- net VDDA_0V75_S0: now also C237.1, U201.8 (NLDO5); no longer C239.1, U201.11 (NLDO3)
- net VDDA_0V85_S0: now also C238.1, U201.10 (NLDO4); no longer C240.1, U201.12 (NLDO2)
- net VDDA_DDR_PLL_S0: now also C240.1, U201.12 (NLDO2); no longer C237.1, U201.8 (NLDO5)
- net VDDQ_DDR_S0: now also C223.1, C224.1, L206.2, R207.2, U201.30 (VOUT6); no longer C235.1, C236.1, L210.2, U201.25 (VOUT10)
- net VDD_CPU_LIT_S0: now also C212.1, C213.1, C214.1, L203.2, U201.56 (VOUT3); no longer C220.1, C221.1, L205.2, R205.2, U201.46 (VOUT5)
- net VDD_DDR_S0: now also C235.1, C236.1, L210.2, U201.25 (VOUT10); no longer C223.1, C224.1, L206.2, R207.2, U201.30 (VOUT6)
- net VDD_GPU_S0: now also C220.1, C221.1, L205.2, R205.2, U201.46 (VOUT5); no longer C216.1, C217.1, C218.1, L204.2, U201.24 (VOUT4)
- net VDD_LOGIC_S0: now also C226.1, C227.1, L207.2, U201.41 (VOUT7); no longer C212.1, C213.1, C214.1, L203.2, U201.56 (VOUT3)
Other:
- moved on the sheet: C201, C207, C211, C212, C213, C214, C215, C219, C220, C221, C222, C223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
