File: hardware/sbc-rk3576/kicad/06_lpddr5.kicad_sch (KiCad schematic)
At the start: 38 parts, among them U401 RK3576, U601 LPDDR5 4GB

Commit message: hardware: add GbE, USB hub + 2x USB-A, Wi-Fi5/BT; real RK3576 land pattern; 100x72 board
- RK3576 footprint from LCSC C42388007 (all 698 ball IDs verified against the
  datasheet) replaces the placeholder.
- RTL8211F-CG RGMII PHY + HR911130C MagJack, FE1.1s 4-port hub (pinout per
  Terminus datasheet), stacked dual USB-A, BL-M8821CU1 Wi-Fi 5/BT 4.2 + u.FL.
- LCSC footprints get pad-derived courtyards; RJ45 pegs become NPTH.
- ERC 0/0, DRC 0 violations, parity 0 (placement stage).

Co-Authored-By: Claude Opus 5.5 <noreply@anthropic.com>
Claude-Session: https://claude.ai/code/session_01DP7VBm9fUdwhcDWq3gWKJ6
Parts:
- U401: footprint sbc:RK3576_FCCSP-698_16.1x17.2mm_PLACEHOLDER -> sbc:RK3576_FCCSP-698_16.1x17.2mm
Changed lines of the file:
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@@
     (property "Reference" "U401" (at 175.26 33.02 0) (effects (font (size 1.27 1.27))))
     (property "Value" "RK3576" (at 175.26 144.78 0) (effects (font (size 1.27 1.27))))
-    (property "Footprint" "sbc:RK3576_FCCSP-698_16.1x17.2mm_PLACEHOLDER"
+    (property "Footprint" "sbc:RK3576_FCCSP-698_16.1x17.2mm"
       (at 175.26 88.9 0)
       (effects (font (size 1.27 1.27)) hide)
