File: hardware/sbc-rk3576/kicad/10_usb.kicad_sch (KiCad schematic)
At the start: 13 parts, among them J1001 USB3.0 A, U1001 USBLC6-2SC6, U1002 TPD4E05U06, U1003 USBLC6-2SC6, U1004 AP2171W

Commit message: hardware: add GbE, USB hub + 2x USB-A, Wi-Fi5/BT; real RK3576 land pattern; 100x72 board
- RK3576 footprint from LCSC C42388007 (all 698 ball IDs verified against the
  datasheet) replaces the placeholder.
- RTL8211F-CG RGMII PHY + HR911130C MagJack, FE1.1s 4-port hub (pinout per
  Terminus datasheet), stacked dual USB-A, BL-M8821CU1 Wi-Fi 5/BT 4.2 + u.FL.
- LCSC footprints get pad-derived courtyards; RJ45 pegs become NPTH.
- ERC 0/0, DRC 0 violations, parity 0 (placement stage).

Co-Authored-By: Claude Opus 5.5 <noreply@anthropic.com>
Claude-Session: https://claude.ai/code/session_01DP7VBm9fUdwhcDWq3gWKJ6
Other:
- note added: "10_usb: USB-C OTG (maskrom) + USB 3.0 host port"
- note removed: "10_usb: USB-C OTG (maskrom) + USB 3.0 host"
- title: USB-C OTG (maskrom) + USB 3.0 host -> USB-C OTG (maskrom) + USB 3.0 host port
Changed lines of the file:
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@@
   (paper "A4")
   (title_block
-    (title "USB-C OTG (maskrom) + USB 3.0 host")
+    (title "USB-C OTG (maskrom) + USB 3.0 host port")
     (date "2026-10-04")
     (rev "A0-draft")
@@
     )
   )
-  (text "10_usb: USB-C OTG (maskrom) + USB 3.0 host"
+  (text "10_usb: USB-C OTG (maskrom) + USB 3.0 host port"
     (at 20 20 0)
     (effects (font (size 3 3)) (justify left bottom))
