File: hardware/sbc-rk3576/kicad/rk3576-sbc.kicad_sch (KiCad schematic)
At the start: 0 parts

Commit message: hardware: add GbE, USB hub + 2x USB-A, Wi-Fi5/BT; real RK3576 land pattern; 100x72 board
- RK3576 footprint from LCSC C42388007 (all 698 ball IDs verified against the
  datasheet) replaces the placeholder.
- RTL8211F-CG RGMII PHY + HR911130C MagJack, FE1.1s 4-port hub (pinout per
  Terminus datasheet), stacked dual USB-A, BL-M8821CU1 Wi-Fi 5/BT 4.2 + u.FL.
- LCSC footprints get pad-derived courtyards; RJ45 pegs become NPTH.
- ERC 0/0, DRC 0 violations, parity 0 (placement stage).

Co-Authored-By: Claude Opus 5.5 <noreply@anthropic.com>
Claude-Session: https://claude.ai/code/session_01DP7VBm9fUdwhcDWq3gWKJ6
Other:
- added sheet 13_ethernet (13_ethernet.kicad_sch)
- added sheet 14_usb_hub_wifi (14_usb_hub_wifi.kicad_sch)
- note added: "Gigabit Ethernet (RTL8211F RGMII)"
- note added: "USB 2.0 hub, 2x USB-A, Wi-Fi 5 + BT module"
- note added: "USB-C OTG (maskrom) + USB 3.0 host port"
- note removed: "USB-C OTG (maskrom) + USB 3.0 host"
Changed lines of the file:
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@@
     (instances (project "rk3576-sbc" (path "/3461ca5d-73ab-5b55-b754-dceefbd02664" (page "11"))))
   )
-  (text "USB-C OTG (maskrom) + USB 3.0 host"
+  (text "USB-C OTG (maskrom) + USB 3.0 host port"
     (at 163 177 0)
     (effects (font (size 1.8 1.8)) (justify left))
@@
     (effects (font (size 1.8 1.8)) (justify left))
   )
+  (sheet
+    (at 290 50)
+    (size 100 25)
+    (fields_autoplaced)
+    (stroke (width 0.1524) (type solid))
+    (fill (color 0 0 0 0))
+    (property "Sheetname" "13_ethernet"
+      (at 290 49.3 0)
+      (effects (font (size 1.27 1.27)) (justify left bottom))
+    )
+    (property "Sheetfile" "13_ethernet.kicad_sch"
+      (at 290 75.6 0)
+      (effects (font (size 1.27 1.27)) (justify left top))
+    )
+    (instances (project "rk3576-sbc" (path "/3461ca5d-73ab-5b55-b754-dceefbd02664" (page "14"))))
+  )
+  (text "Gigabit Ethernet (RTL8211F RGMII)"
+    (at 293 63 0)
+    (effects (font (size 1.8 1.8)) (justify left))
+  )
+  (sheet
+    (at 290 88)
+    (size 100 25)
+    (fields_autoplaced)
+    (stroke (width 0.1524) (type solid))
+    (fill (color 0 0 0 0))
+    (property "Sheetname" "14_usb_hub_wifi"
+      (at 290 87.3 0)
+      (effects (font (size 1.27 1.27)) (justify left bottom))
+    )
+    (property "Sheetfile" "14_usb_hub_wifi.kicad_sch"
+      (at 290 113.6 0)
+      (effects (font (size 1.27 1.27)) (justify left top))
+    )
+    (instances (project "rk3576-sbc" (path "/3461ca5d-73ab-5b55-b754-dceefbd02664" (page "15"))))
+  )
+  (text "USB 2.0 hub, 2x USB-A, Wi-Fi 5 + BT module"
+    (at 293 101 0)
+    (effects (font (size 1.8 1.8)) (justify left))
+  )
